File: pcb/holocube_transfer_board/holocube_transfer_board.kicad_pcb (KiCad board)
At the start: 2 copper layers, 51.5 x 32 mm, 3 parts, among them J1 Conn_01x15_Female, J2 Conn_01x15_Female, J3 Conn_01x08_Female

Commit message: update holocude_transfer_board
Connections:
- J1 pad 4: Net-(J1-Pad4) -> unconnected-(J1-Pad4)
- J1 pad 5: unconnected-(J1-Pad5) -> Net-(J3-Pad8)
- J3 pad 8: Net-(J1-Pad4) -> Net-(J3-Pad8)
Routing:
- net Net-(J3-Pad8): track 0.00 -> 12.5 mm
- net Net-(J1-Pad4): track 9.97 -> 0.00 mm
Changed lines of the file:
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@@
   (net 2 "Net-(J1-Pad2)")
   (net 3 "unconnected-(J1-Pad3)")
-  (net 4 "Net-(J1-Pad4)")
-  (net 5 "unconnected-(J1-Pad5)")
+  (net 4 "unconnected-(J1-Pad4)")
+  (net 5 "Net-(J3-Pad8)")
   (net 6 "unconnected-(J1-Pad6)")
   (net 7 "unconnected-(J1-Pad7)")
@@
       (net 8 "Net-(J1-Pad8)") (pinfunction "Pin_7") (pintype "passive"))
     (pad "8" thru_hole oval locked (at 0 17.78 180) (size 1.7 1.7) (drill 1) (layers *.Cu *.Mask)
-      (net 4 "Net-(J1-Pad4)") (pinfunction "Pin_8") (pintype "passive"))
+      (net 5 "Net-(J3-Pad8)") (pinfunction "Pin_8") (pintype "passive"))
     (model "${KICAD6_3DMODEL_DIR}/Connector_PinSocket_2.54mm.3dshapes/PinSocket_1x08_P2.54mm_Vertical.wrl"
       (offset (xyz 0 0 0))
@@
       (net 3 "unconnected-(J1-Pad3)") (pinfunction "Pin_3") (pintype "passive"))
     (pad "4" thru_hole oval locked (at 0 -7.62 270) (size 1.7 1.7) (drill 1) (layers *.Cu *.Mask)
-      (net 4 "Net-(J1-Pad4)") (pinfunction "Pin_4") (pintype "passive"))
+      (net 4 "unconnected-(J1-Pad4)") (pinfunction "Pin_4") (pintype "passive"))
     (pad "5" thru_hole oval locked (at 0 -10.16 270) (size 1.7 1.7) (drill 1) (layers *.Cu *.Mask)
-      (net 5 "unconnected-(J1-Pad5)") (pinfunction "Pin_5") (pintype "passive"))
+      (net 5 "Net-(J3-Pad8)") (pinfunction "Pin_5") (pintype "passive"))
     (pad "6" thru_hole oval locked (at 0 -12.7 270) (size 1.7 1.7) (drill 1) (layers *.Cu *.Mask)
       (net 6 "unconnected-(J1-Pad6)") (pinfunction "Pin_6") (pintype "passive"))
@@
   (segment (start 121.49 114) (end 116.28 108.79) (width 0.25) (layer "B.Cu") (net 2))
   (segment (start 116.28 108.79) (end 116.28 98.3) (width 0.25) (layer "B.Cu") (net 2))
-  (segment (start 117.565 102.095) (end 121.36 98.3) (width 0.25) (layer "F.Cu") (net 4))
-  (segment (start 112.965 102.095) (end 117.565 102.095) (width 0.25) (layer "F.Cu") (net 4))
+  (segment (start 112.965 102.095) (end 120.105 102.095) (width 0.25) (layer "F.Cu") (net 5))
+  (segment (start 120.105 102.095) (end 123.9 98.3) (width 0.25) (layer "F.Cu") (net 5))
   (segment (start 112.965 104.635) (end 125.185 104.635) (width 0.25) (layer "F.Cu") (net 8))
   (segment (start 125.185 104.635) (end 131.52 98.3) (width 0.25) (layer "F.Cu") (net 8))
