File: pcb/holocube_transfer_board/holocube_transfer_board.kicad_sch (KiCad schematic)
At the start: 3 parts, among them J1 Conn_01x15_Female, J2 Conn_01x15_Female, J3 Conn_01x08_Female

Commit message: update holocude_transfer_board
Connections:
- net at J3.8 (Pin_8): now also J1.5 (Pin_5); no longer J1.4 (Pin_4)
Changed lines of the file:
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@@
+    (stroke (width 0) (type default) (color 0 0 0 0))
+  )
+  (wire (pts (xy 129.54 77.47) (xy 129.54 111.76))
     (stroke (width 0) (type default) (color 0 0 0 0))
   )
@@
     (stroke (width 0) (type default) (color 0 0 0 0))
   )
-  (wire (pts (xy 129.54 74.93) (xy 129.54 111.76))
-    (stroke (width 0) (type default) (color 0 0 0 0))
-  )
   (wire (pts (xy 114.3 111.76) (xy 114.3 67.31))
     (stroke (width 0) (type default) (color 0 0 0 0))
@@
     (stroke (width 0) (type default) (color 0 0 0 0))
   )
-  (wire (pts (xy 100.33 74.93) (xy 129.54 74.93))
-    (stroke (width 0) (type default) (color 0 0 0 0))
-  )
   (wire (pts (xy 124.46 92.71) (xy 124.46 111.76))
     (stroke (width 0) (type default) (color 0 0 0 0))
   )
+  (wire (pts (xy 100.33 77.47) (xy 129.54 77.47))
+    (stroke (width 0) (type default) (color 0 0 0 0))
+  )
